Commit message: Depth integration

File: x3_sim/urdf/x3.ign.xacro (robot description, xacro)
@@ -87,5 +87,5 @@
           name="ignition::gazebo::systems::MulticopterVelocityControl">
           <robotNamespace>${robot_namespace}</robotNamespace>
-          <commandSubTopic>gazebo/command/twist</commandSubTopic>
+          <commandSubTopic>cmd_vel</commandSubTopic>
           <enableSubTopic>enable</enableSubTopic>
           <comLinkName>${robot_namespace}/base_footprint</comLinkName>
@@ -125,9 +125,30 @@
           name="ignition::gazebo::systems::OdometryPublisher">
           <dimensions>3</dimensions>
+          <topic>${robot_namespace}/odom</topic>
         </plugin>
         <plugin
           filename="ignition-gazebo-joint-state-publisher-system"
           name="ignition::gazebo::systems::JointStatePublisher">
+          <topic>${robot_namespace}/joint_states</topic>
         </plugin>
+    </gazebo>
+    <gazebo reference='${robot_namespace}/base_footprint'>
+        <sensor name="camera_front" type="rgbd_camera">
+          <topic>${robot_namespace}/camera</topic>
+          <camera name="camera_front">
+            <horizontal_fov>1.05</horizontal_fov>
+            <image>
+              <width>256</width>
+              <height>256</height>
+            </image>
+            <clip>
+              <near>0.1</near>
+              <far>10.0</far>
+            </clip>
+          </camera>
+          <always_on>1</always_on>
+          <update_rate>20</update_rate>
+          <visualize>0</visualize>
+        </sensor>
     </gazebo>
   </xacro:macro>

File: x3_sim/urdf/x3.xacro (robot description, xacro)
@@ -113,4 +113,10 @@
       </visual>
     </link>
+    <link name='${robot_namespace}/camera_link' />
+    <joint name='${robot_namespace}/camera_joint' type='fixed'>
+      <parent link='${robot_namespace}/base_link'/>
+      <child link='${robot_namespace}/camera_link'/>
+      <origin xyz='0.12 0 0' rpy='0 0 0'/>
+    </joint>
     <joint name='${robot_namespace}/base_joint' type='fixed'>
       <parent link='${robot_namespace}/base_footprint'/>
